Commit message: The robot only has HFE joints move. Other joints are fixed successfully

File: ksluck_sim_private/pybullet_ksluck/data/anymal_flat/urdf/anymal_basic.urdf (robot description, URDF)
Before this commit: robot anymal, 18 links, 17 joints
Joints:
- joint LF_HAA: axis 1 0 0 -> 0 0 0; type revolute -> fixed
- joint LF_KFE: axis 0 1 0 -> 0 0 0; type revolute -> fixed
- joint LH_HAA: axis 1 0 0 -> 0 0 0; type revolute -> fixed
- joint LH_KFE: axis 0 1 0 -> 0 0 0; type revolute -> fixed
- joint RF_HAA: axis 1 0 0 -> 0 0 0; type revolute -> fixed
- joint RF_KFE: axis 0 1 0 -> 0 0 0; type revolute -> fixed
- joint RH_HAA: axis 1 0 0 -> 0 0 0; type revolute -> fixed
- joint RH_KFE: axis 0 1 0 -> 0 0 0; type revolute -> fixed

Commit message: changed the range of HAA and HFE.

File: ksluck_sim_private/pybullet_ksluck/data/anymal_flat/urdf/anymal_basic.urdf (robot description, URDF)
Before this commit: robot anymal, 18 links, 17 joints
Joints:
- joint LF_HAA: axis 0 0 0 -> 1 0 0; limit lower=-6.28 upper=6.28 effort=80 velocity=15 -> lower=-0.35 upper=0.35 effort=80 velocity=15; type fixed -> revolute
- joint LF_HFE: limit lower=-6.28 upper=6.28 effort=80 velocity=15 -> lower=-0.8 upper=0.8 effort=80 velocity=15
- joint LH_HAA: axis 0 0 0 -> 1 0 0; limit lower=-6.28 upper=6.28 effort=80 velocity=15 -> lower=-0.35 upper=0.35 effort=80 velocity=15; type fixed -> revolute
- joint LH_HFE: limit lower=-6.28 upper=6.28 effort=80 velocity=15 -> lower=-0.8 upper=0.8 effort=80 velocity=15
- joint RF_HAA: axis 0 0 0 -> 1 0 0; limit lower=-6.28 upper=6.28 effort=80 velocity=15 -> lower=-0.35 upper=0.35 effort=80 velocity=15; type fixed -> revolute
- joint RF_HFE: limit lower=-6.28 upper=6.28 effort=80 velocity=15 -> lower=-0.8 upper=0.8 effort=80 velocity=15
- joint RH_HAA: axis 0 0 0 -> 1 0 0; limit lower=-6.28 upper=6.28 effort=80 velocity=15 -> lower=-0.35 upper=0.35 effort=80 velocity=15; type fixed -> revolute
- joint RH_HFE: limit lower=-6.28 upper=6.28 effort=80 velocity=15 -> lower=-0.8 upper=0.8 effort=80 velocity=15

Commit message: anymal is now restricted to x plane

File: ksluck_sim_private/pybullet_ksluck/data/anymal_flat/urdf/anymal_basic.urdf (robot description, URDF)
Before this commit: robot anymal, 18 links, 17 joints
Links:
- added link anymal
- added link world
- added link world_2
- added link world_3
Joints:
- added joint ignore_anymal: type fixed, parent base, child anymal, origin xyz=0 0 0  rpy=0 0 0, axis 0 1 0
- added joint ignore_ignore_world_y: type revolute, parent world_2, child world_3, origin xyz=0 0 0  rpy=0 0 0, axis 0 1 0, limit lower=-360 upper=360
- added joint ignore_world_x: type prismatic, parent world, child world_2, origin xyz=0 0 0  rpy=0 0 0, axis 1 0 0, limit lower=-10000000 upper=10000000
- added joint ignore_world_z: type prismatic, parent world_3, child base, origin xyz=0 0 0  rpy=0 0 0, axis 0 0 1, limit lower=-10000000 upper=10000000

Commit message: Did some tuning

File: ksluck_sim_private/pybullet_ksluck/data/anymal_flat/urdf/anymal_basic.urdf (robot description, URDF)
Before this commit: robot anymal, 18 links, 17 joints
Joints:
- joint LF_KFE: axis 0 0 0 -> 0 1 0; limit lower=-6.28 upper=6.28 effort=80 velocity=15 -> lower=-0.35 upper=0.35 effort=80 velocity=15; type fixed -> revolute
- joint LH_KFE: axis 0 0 0 -> 0 1 0; limit lower=-6.28 upper=6.28 effort=80 velocity=15 -> lower=-0.35 upper=0.35 effort=80 velocity=15; type fixed -> revolute
- joint RF_KFE: axis 0 0 0 -> 0 1 0; limit lower=-6.28 upper=6.28 effort=80 velocity=15 -> lower=-0.35 upper=0.35 effort=80 velocity=15; type fixed -> revolute
- joint RH_KFE: axis 0 0 0 -> 0 1 0; limit lower=-6.28 upper=6.28 effort=80 velocity=15 -> lower=-0.35 upper=0.35 effort=80 velocity=15; type fixed -> revolute
